File: hardware/g660-ctrl.kicad_pcb (KiCad board)
At the start: 4 copper layers, 36.3 x 60.5 mm, 51 parts, among them J2 USB_C, J3 GPIO, J4 BATTERY, J5 JST PH - I2C, J6 JST PH - UART1, J7 JST PH - UART2, J8 DIFF_CONN, M1 DIFF, Q1 Dual_Q_PMOS_SGD, Q2 2N7002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

Commit message: feat: Complete G660 control board
Parts:
- DIFF POS: renamed from J8
- renumbered SW7 to BOOT, J5 to I2C, SW8 to RST, J6 to TX1
Changed lines of the file:
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@@
 			(outputformat 1)
 			(mirror no)
-			(drillshape 1)
+			(drillshape 0)
 			(scaleselection 1)
-			(outputdirectory "")
+			(outputdirectory "../fabrication/")
 		)
 	)
@@
 		(descr "https://katalog.we-online.com/em/datasheet/434133025816.pdf")
 		(tags "tactile switch Wurth Wuerth")
-		(property "Reference" "SW7"
+		(property "Reference" "BOOT"
 			(at 0.15 -3.429 0)
 			(layer "F.SilkS" knockout)
@@
 		(layer "F.Cu")
 		(at 162.771 94.674 -90)
-		(property "Reference" "J8"
-			(at -0.127 2.286 -90)
+		(property "Reference" "DIFF POS"
+			(at -0.127 2.286 270)
 			(unlocked yes)
 			(layer "B.SilkS" knockout)
@@
 		(layer "F.Cu")
 		(at 136.482 94.293 -90)
-		(property "Reference" "J5"
+		(property "Reference" "I2C"
 			(at 0 2.159 270)
 			(unlocked yes)
@@
 		(layer "F.Cu")
 		(at 143.721 85.149)
-		(property "Reference" "J6"
-			(at -1.27 3.60681 -90)
+		(property "Reference" "TX1"
+			(at -1.27 3.60681 270)
 			(unlocked yes)
 			(layer "B.SilkS" knockout)
@@
 		(descr "https://katalog.we-online.com/em/datasheet/434133025816.pdf")
 		(tags "tactile switch Wurth Wuerth")
-		(property "Reference" "SW8"
+		(property "Reference" "RST"
 			(at -0.038 -3.429 0)
 			(layer "F.SilkS" knockout)
